File: myck_pcb/myck_pcb.kicad_sch (KiCad schematic)
At the start: 92 parts, among them M1 SW_Push_45deg, M2 SW_Push_45deg

Commit message: Creado esquema PCB
La PCB inicial, como es una prueba, sólo va a tener 4 teclas.
Empezando a añadir RGB-leds
Parts:
- added LED1, LED2, LED3, LED4: MX_SK6812MINI-E, PCM_marbastlib-mx:LED_MX_6028R, symbol PCM_marbastlib-mx:MX_SK6812MINI-E
- -1: renamed from -; footprint (none) -> PCM_marbastlib-xp-gateron_lp:SW_KS33_HS_KS-2P02B01-02_HS_1u
- A1: renamed from A; footprint (none) -> PCM_marbastlib-xp-gateron_lp:SW_KS33_HS_KS-2P02B01-02_HS_1u
- Alt-l1: renamed from Alt-l; footprint (none) -> PCM_marbastlib-xp-gateron_lp:SW_KS33_HS_KS-2P02B01-02_HS_1u
- Alt-r1: renamed from Alt-r; footprint (none) -> PCM_marbastlib-xp-gateron_lp:SW_KS33_HS_KS-2P02B01-02_HS_1u
- B1: renamed from B; footprint (none) -> PCM_marbastlib-xp-gateron_lp:SW_KS33_HS_KS-2P02B01-02_HS_1u
- BackSpace1: renamed from BackSpace; footprint (none) -> PCM_marbastlib-xp-gateron_lp:SW_KS33_HS_KS-2P02B01-02_HS_1u
- C1: renamed from C; footprint (none) -> PCM_marbastlib-xp-gateron_lp:SW_KS33_HS_KS-2P02B01-02_HS_1u
- CapsLock1: renamed from CapsLock; footprint (none) -> PCM_marbastlib-xp-gateron_lp:SW_KS33_HS_KS-2P02B01-02_HS_1u
- Comma1: renamed from Comma; footprint (none) -> PCM_marbastlib-xp-gateron_lp:SW_KS33_HS_KS-2P02B01-02_HS_1u
- Ctrl-l1: renamed from Ctrl-l; footprint (none) -> PCM_marbastlib-xp-gateron_lp:SW_KS33_HS_KS-2P02B01-02_HS_1u
- Ctrl-r1: renamed from Ctrl-r; footprint (none) -> PCM_marbastlib-xp-gateron_lp:SW_KS33_HS_KS-2P02B01-02_HS_1u
- D1, D10, D11, D12, D13, D14, D15, D16, D17, D18, D19, D2, D20, D21, D22, D23, D24, D25, D26, D27, D28, D29, D3, D30, D31, D32, D33, D34, D35, D36, D37, D38, D39, D4, D40, D41, D42, D43, D44, D45, D46, D5, D6, D7, D8, D9: footprint (none) -> Diode_SMD:D_SOD-123
- D47: renamed from D; footprint (none) -> PCM_marbastlib-xp-gateron_lp:SW_KS33_HS_KS-2P02B01-02_HS_1u
- Dot1: renamed from Dot; footprint (none) -> PCM_marbastlib-xp-gateron_lp:SW_KS33_HS_KS-2P02B01-02_HS_1u
- E1: renamed from E; footprint (none) -> PCM_marbastlib-xp-gateron_lp:SW_KS33_HS_KS-2P02B01-02_HS_1u
- Enter1: renamed from Enter; footprint (none) -> PCM_marbastlib-xp-gateron_lp:SW_KS33_HS_KS-2P02B01-02_HS_1u
- F1: renamed from F; footprint (none) -> PCM_marbastlib-xp-gateron_lp:SW_KS33_HS_KS-2P02B01-02_HS_1u
- G1: renamed from G; footprint (none) -> PCM_marbastlib-xp-gateron_lp:SW_KS33_HS_KS-2P02B01-02_HS_1u
- H1: renamed from H; footprint (none) -> PCM_marbastlib-xp-gateron_lp:SW_KS33_HS_KS-2P02B01-02_HS_1u
- I1: renamed from I; footprint (none) -> PCM_marbastlib-xp-gateron_lp:SW_KS33_HS_KS-2P02B01-02_HS_1u
- J1: renamed from J; footprint (none) -> PCM_marbastlib-xp-gateron_lp:SW_KS33_HS_KS-2P02B01-02_HS_1u
- K1: renamed from K; footprint (none) -> PCM_marbastlib-xp-gateron_lp:SW_KS33_HS_KS-2P02B01-02_HS_1u
- L1: renamed from L; footprint (none) -> PCM_marbastlib-xp-gateron_lp:SW_KS33_HS_KS-2P02B01-02_HS_1u
- M1, M2: footprint (none) -> PCM_marbastlib-xp-gateron_lp:SW_KS33_HS_KS-2P02B01-02_HS_1u
- M3: renamed from M; footprint (none) -> PCM_marbastlib-xp-gateron_lp:SW_KS33_HS_KS-2P02B01-02_HS_1u
- N1: renamed from N; footprint (none) -> PCM_marbastlib-xp-gateron_lp:SW_KS33_HS_KS-2P02B01-02_HS_1u
- O1: renamed from O; footprint (none) -> PCM_marbastlib-xp-gateron_lp:SW_KS33_HS_KS-2P02B01-02_HS_1u
- P1: renamed from P; footprint (none) -> PCM_marbastlib-xp-gateron_lp:SW_KS33_HS_KS-2P02B01-02_HS_1u
- Q1: renamed from Q; footprint (none) -> PCM_marbastlib-xp-gateron_lp:SW_KS33_HS_KS-2P02B01-02_HS_1u
- R1: renamed from R; footprint (none) -> PCM_marbastlib-xp-gateron_lp:SW_KS33_HS_KS-2P02B01-02_HS_1u
- S1: renamed from S; footprint (none) -> PCM_marbastlib-xp-gateron_lp:SW_KS33_HS_KS-2P02B01-02_HS_1u
- Shift-l1: renamed from Shift-l; footprint (none) -> PCM_marbastlib-xp-gateron_lp:SW_KS33_HS_KS-2P02B01-02_HS_1u
- Shift-r1: renamed from Shift-r; footprint (none) -> PCM_marbastlib-xp-gateron_lp:SW_KS33_HS_KS-2P02B01-02_HS_1u
- Space-l1: renamed from Space-l; footprint (none) -> PCM_marbastlib-xp-gateron_lp:SW_KS33_HS_KS-2P02B01-02_HS_1u
- Space-r1: renamed from Space-r; footprint (none) -> PCM_marbastlib-xp-gateron_lp:SW_KS33_HS_KS-2P02B01-02_HS_1u
- Super-l1: renamed from Super-l; footprint (none) -> PCM_marbastlib-xp-gateron_lp:SW_KS33_HS_KS-2P02B01-02_HS_1u
- Super-r1: renamed from Super-r; footprint (none) -> PCM_marbastlib-xp-gateron_lp:SW_KS33_HS_KS-2P02B01-02_HS_1u
- T1: renamed from T; footprint (none) -> PCM_marbastlib-xp-gateron_lp:SW_KS33_HS_KS-2P02B01-02_HS_1u
- Tab1: renamed from Tab; footprint (none) -> PCM_marbastlib-xp-gateron_lp:SW_KS33_HS_KS-2P02B01-02_HS_1u
- Tilde1: renamed from Tilde; footprint (none) -> PCM_marbastlib-xp-gateron_lp:SW_KS33_HS_KS-2P02B01-02_HS_1u
- U1: renamed from U; footprint (none) -> PCM_marbastlib-xp-gateron_lp:SW_KS33_HS_KS-2P02B01-02_HS_1u
- V1: renamed from V; footprint (none) -> PCM_marbastlib-xp-gateron_lp:SW_KS33_HS_KS-2P02B01-02_HS_1u
- W1: renamed from W; footprint (none) -> PCM_marbastlib-xp-gateron_lp:SW_KS33_HS_KS-2P02B01-02_HS_1u
- X1: renamed from X; footprint (none) -> PCM_marbastlib-xp-gateron_lp:SW_KS33_HS_KS-2P02B01-02_HS_1u
- Y1: renamed from Y; footprint (none) -> PCM_marbastlib-xp-gateron_lp:SW_KS33_HS_KS-2P02B01-02_HS_1u
- Z1: renamed from Z; footprint (none) -> PCM_marbastlib-xp-gateron_lp:SW_KS33_HS_KS-2P02B01-02_HS_1u
Connections:
- new net: LED2.2 (DOUT), LED3.3 (DIN)
- new net: LED1.2 (DOUT), LED2.3 (DIN)
- new net: LED3.2 (DOUT), LED4.3 (DIN)
- new net RGB: LED1.3 (DIN)
- no-connect marks 0 -> 1

Commit message: Añadidos Leds, circuitos y pines
En principio, creo que ya estaría la circuitería hecha.
Connections:
- net +5V: now reaches LED2.1 (VDD)
- net +5V: now also LED1.1 (VDD), LED3.1 (VDD), LED4.1 (VDD)
- net Earth: now reaches LED2.4 (VSS)
- net Earth: now also LED1.4 (VSS), LED3.4 (VSS), LED4.4 (VSS)
